Commit message: 跑通sim2sim

File: bike_rl_sim2sim2real/src/tita_locomotion/tita_description/bike/urdf/robot.urdf (robot description, URDF)
Before this commit: robot bike250311, 4 links, 3 joints
Links:
- added link imu_link, mass 0.001; collision box size=.001 .001 .001; visual box size=0.001 0.001 0.001
Joints:
- added joint imu_joint: type fixed, parent base_link, child imu_link, origin xyz=0 0 0 rpy=0 0 0
- joint joint_f_wheel: limit lower=-10000 upper=10000 effort=30 velocity=200 -> lower=-10000 upper=10000 effort=100 velocity=200
- joint joint_front_turn: limit lower=-1.3 upper=1.3 effort=20 velocity=12.5 -> lower=-1.3 upper=1.3 effort=100 velocity=12.5
- joint joint_rear_wheel: limit lower=-1000000 upper=10000000 effort=30 velocity=200 -> lower=-1000000 upper=10000000 effort=100 velocity=200

File: bike_rl_sim2sim2real/src/tita_locomotion/tita_description/bike/xacro/description.xacro (robot description, xacro)
@@ -119,5 +119,5 @@
       <axis
         xyz="0 0 -1" />
-      <limit effort="20" lower="-1.3" upper="1.3" velocity="12.5"/>
+      <limit effort="100" lower="-1.3" upper="1.3" velocity="12.5"/>
     </joint>
     <link
@@ -172,5 +172,5 @@
       <axis
         xyz="0 0 1" />
-      <limit effort="30" lower="-10000" upper="10000" velocity="200"/>
+      <limit effort="100" lower="-10000" upper="10000" velocity="200"/>
     </joint>
     <link
@@ -225,5 +225,5 @@
       <axis
         xyz="0 0 -1" />
-      <limit effort="30" lower="-1000000" upper="10000000" velocity="200"/>
+      <limit effort="100" lower="-1000000" upper="10000000" velocity="200"/>
     </joint>
   </xacro:macro>

Commit message: 修改小问题并且尝试使用参数文件

File: bike_rl_sim2sim2real/src/tita_locomotion/tita_description/bike/urdf/robot.urdf (robot description, URDF)
Before this commit: robot bike, 5 links, 4 joints
Links:
- link front_wheel: geometry collision mesh filename=../meshes/front_wheel.STL; visual mesh filename=../meshes/front_wheel.STL
- link rear_wheel: geometry collision mesh filename=../meshes/rear_wheel.STL; visual mesh filename=../meshes/rear_wheel.STL

File: bike_rl_sim2sim2real/src/tita_locomotion/tita_description/bike/xacro/description.xacro (robot description, xacro)
@@ -156,5 +156,6 @@
           rpy="0 0 0" />
         <geometry>
-          <cylinder length="0.05" radius="0.33"/>
+          <mesh
+            filename="../meshes/front_wheel.STL" />
         </geometry>
       </collision>
@@ -209,5 +210,6 @@
           rpy="0 0 0" />
         <geometry>
-          <cylinder length="0.05" radius="0.33"/>
+          <mesh
+            filename="../meshes/rear_wheel.STL" />
         </geometry>
       </collision>
