Commit message: more bike modules and controller

File: bike_rl_sim2sim2real/src/tita_locomotion/tita_description/bike/xacro/robot.xacro (robot description, xacro)
@@ -2,4 +2,5 @@
 <robot xmlns:xacro="http://wiki.ros.org/xacro" name="bike">
   <xacro:arg name="prefix" default="" />
+  <xacro:arg name="use_heavy" default="false" />
   <xacro:property name="sim_env" value="$(arg sim_env)" />
   <xacro:property name="ctrl_mode" value="$(arg ctrl_mode)" />
@@ -7,4 +8,14 @@
   <xacro:include filename="$(find tita_description)/bike/xacro/materials.xacro" />
   <xacro:include filename="$(find tita_description)/bike/xacro/description.xacro" />
+  <xacro:if value="$(arg use_heavy)">
+    <xacro:include filename="$(find tita_description)/bike/xacro/heavy.xacro" />
+      <joint name="joint_heavy" type="fixed">
+        <origin xyz="0.1 0 0.13" rpy="0 0 0" />
+        <parent link="base_link" />
+        <child link="heavy_link" />
+        <axis xyz="0 0 0" />
+      </joint>
+    <xacro:bike_heavy />
+  </xacro:if>
   <xacro:include filename="$(find tita_description)/bike/xacro/ros2control.xacro" />
   <xacro:if value="${sim_env == 'none'}">
