Commit message: 硬件测试

File: bike_rl_sim2sim2real/src/tita_locomotion/tita_description/bikeR/xacro/ros2control.xacro (robot description, xacro)
@@ -58,4 +58,19 @@
         </xacro:if>
       </hardware>
+      <joint name="joint_front_dummy">
+        <command_interface name="position"/>
+        <command_interface name="velocity"/>
+        <command_interface name="effort">
+          <param name="min">-20</param>
+          <param name="max">20</param>
+        </command_interface>
+        <command_interface name="kp"/>
+        <command_interface name="kd"/>
+        <state_interface name="position">
+          <param name="initial_value">0.0</param>
+        </state_interface>
+        <state_interface name="velocity"/>
+        <state_interface name="effort"/>
+      </joint>
       <joint name="joint_front_turn">
         <command_interface name="position"/>
